File: kicad/v2_numpad/esp32.kicad_sch (KiCad schematic)
At the start: 3 parts, among them U1 ESP32-S3-WROOM-1-N16R8

Commit message: [kicad] some more minor tweaks to the numpad
Parts:
- added U3: AMS1117-3.3, Package_TO_SOT_SMD:SOT-223-3_TabPin2, symbol Regulator_Linear:AMS1117-3.3
- C6: value C -> 10uF/25V (20%)
- C7: value C -> .1uF/50V (10%)
Connections:
- net ESP_3V3: now reaches C7.1
- net ESP_3V3: now also C6.1, U1.2 (3V3)
- net GND: now reaches C7.2
- net GND: now also C6.2, U1.1 (GND)
Other:
- moved on the sheet: C6, C7
Changed lines of the file:
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@@
     (title "ESP32")
   )
-  (symbol (lib_id "Device:C") (at 64.77 127 0) (unit 1)
-    (in_bom yes) (on_board yes) (dnp no) (fields_autoplaced)
-    (property "Reference" "C7" (at 68.58 125.73 0)
-      (effects (font (size 1.27 1.27)) (justify left))
-    )
-    (property "Value" "C" (at 68.58 128.27 0)
-      (effects (font (size 1.27 1.27)) (justify left))
-    )
-    (property "Footprint" "" (at 65.7352 130.81 0)
-      (effects (font (size 1.27 1.27)) hide)
-    )
-    (property "Datasheet" "~" (at 64.77 127 0)
+  (junction (at 48.26 43.18) (diameter 0) (color 0 0 0 0)
+  )
+  (junction (at 77.47 31.75) (diameter 0) (color 0 0 0 0)
+  )
+  (junction (at 48.26 31.75) (diameter 0) (color 0 0 0 0)
+  )
+  (junction (at 72.39 31.75) (diameter 0) (color 0 0 0 0)
+  )
+  (wire (pts (xy 72.39 31.75) (xy 77.47 31.75))
+    (stroke (width 0) (type default))
+  )
+  (wire (pts (xy 72.39 39.37) (xy 72.39 43.18))
+    (stroke (width 0) (type default))
+  )
+  (wire (pts (xy 72.39 43.18) (xy 48.26 43.18))
+    (stroke (width 0) (type default))
+  )
+  (wire (pts (xy 48.26 39.37) (xy 48.26 43.18))
+    (stroke (width 0) (type default))
+  )
+  (wire (pts (xy 77.47 31.75) (xy 77.47 22.86))
+    (stroke (width 0) (type default))
+  )
+  (wire (pts (xy 48.26 43.18) (xy 48.26 46.99))
+    (stroke (width 0) (type default))
+  )
+  (wire (pts (xy 48.26 31.75) (xy 72.39 31.75))
+    (stroke (width 0) (type default))
+  )
+  (wire (pts (xy 48.26 22.86) (xy 48.26 31.75))
+    (stroke (width 0) (type default))
+  )
+  (wire (pts (xy 90.17 29.21) (xy 90.17 26.67))
+    (stroke (width 0) (type default))
+  )
+  (wire (pts (xy 92.71 31.75) (xy 77.47 31.75))
+    (stroke (width 0) (type default))
+  )
+  (wire (pts (xy 92.71 29.21) (xy 90.17 29.21))
+    (stroke (width 0) (type default))
+  )
+  (label "VCC_3V3" (at 48.26 22.86 0) (fields_autoplaced)
+    (effects (font (size 1.27 1.27)) (justify left bottom))
+  )
+  (label "ESP_3V3" (at 77.47 22.86 0) (fields_autoplaced)
+    (effects (font (size 1.27 1.27)) (justify left bottom))
+  )
+  (symbol (lib_id "power:GND") (at 90.17 26.67 180) (unit 1)
+    (in_bom yes) (on_board yes) (dnp no) (fields_autoplaced)
+    (property "Reference" "#PWR06" (at 90.17 20.32 0)
+      (effects (font (size 1.27 1.27)) hide)
+    )
+    (property "Value" "GND" (at 90.17 21.59 0)
+      (effects (font (size 1.27 1.27)))
+    )
+    (property "Footprint" "" (at 90.17 26.67 0)
+      (effects (font (size 1.27 1.27)) hide)
+    )
+    (property "Datasheet" "" (at 90.17 26.67 0)
+      (effects (font (size 1.27 1.27)) hide)
+    )
+    (pin "1")
+    (instances
+      (project "v2_numpad"
+        (path "/42eee74c-d04d-4a1d-8e02-a7aca1694734/74c564bf-cb18-45a0-a3d5-47831683800e"
+          (reference "#PWR06") (unit 1)
+        )
+      )
+    )
+  )
+  (symbol (lib_id "Regulator_Linear:AMS1117-3.3") (at 50.8 135.89 0) (unit 1)
+    (in_bom yes) (on_board yes) (dnp no) (fields_autoplaced)
+    (property "Reference" "U3" (at 50.8 129.54 0)
+      (effects (font (size 1.27 1.27)))
+    )
+    (property "Value" "AMS1117-3.3" (at 50.8 132.08 0)
+      (effects (font (size 1.27 1.27)))
+    )
+    (property "Footprint" "Package_TO_SOT_SMD:SOT-223-3_TabPin2" (at 50.8 130.81 0)
+      (effects (font (size 1.27 1.27)) hide)
+    )
+    (property "Datasheet" "http://www.advanced-monolithic.com/pdf/ds1117.pdf" (at 53.34 142.24 0)
+      (effects (font (size 1.27 1.27)) hide)
+    )
+    (property "JLCPCB Part" "C6186" (at 50.8 135.89 0)
+      (effects (font (size 1.27 1.27)) hide)
+    )
+    (pin "1")
+    (pin "2")
+    (pin "3")
+    (instances
+      (project "v2_numpad"
+        (path "/42eee74c-d04d-4a1d-8e02-a7aca1694734/74c564bf-cb18-45a0-a3d5-47831683800e"
+          (reference "U3") (unit 1)
+        )
+      )
+    )
+  )
+  (symbol (lib_id "Device:C") (at 72.39 35.56 0) (unit 1)
+    (in_bom yes) (on_board yes) (dnp no) (fields_autoplaced)
+    (property "Reference" "C7" (at 76.2 34.29 0)
+      (effects (font (size 1.27 1.27)) (justify left))
+    )
+    (property "Value" ".1uF/50V (10%)" (at 76.2 36.83 0)
+      (effects (font (size 1.27 1.27)) (justify left))
+    )
+    (property "Footprint" "" (at 73.3552 39.37 0)
+      (effects (font (size 1.27 1.27)) hide)
+    )
+    (property "Datasheet" "~" (at 72.39 35.56 0)
       (effects (font (size 1.27 1.27)) hide)
     )
@@
     )
   )
-  (symbol (lib_id "Device:C") (at 44.45 127 0) (unit 1)
-    (in_bom yes) (on_board yes) (dnp no) (fields_autoplaced)
-    (property "Reference" "C6" (at 48.26 125.73 0)
-      (effects (font (size 1.27 1.27)) (justify left))
-    )
-    (property "Value" "C" (at 48.26 128.27 0)
-      (effects (font (size 1.27 1.27)) (justify left))
-    )
-    (property "Footprint" "" (at 45.4152 130.81 0)
-      (effects (font (size 1.27 1.27)) hide)
-    )
-    (property "Datasheet" "~" (at 44.45 127 0)
+  (symbol (lib_id "Device:C") (at 48.26 35.56 0) (unit 1)
+    (in_bom yes) (on_board yes) (dnp no)
+    (property "Reference" "C6" (at 52.07 34.29 0)
+      (effects (font (size 1.27 1.27)) (justify left))
+    )
+    (property "Value" "10uF/25V (20%)" (at 52.07 36.83 0)
+      (effects (font (size 1.27 1.27)) (justify left))
+    )
+    (property "Footprint" "" (at 49.2252 39.37 0)
+      (effects (font (size 1.27 1.27)) hide)
+    )
+    (property "Datasheet" "~" (at 48.26 35.56 0)
       (effects (font (size 1.27 1.27)) hide)
     )
@@
     )
   )
-  (symbol (lib_id "mantyl:ESP32-S3-WROOM-1") (at 83.82 60.96 0) (unit 1)
-    (in_bom yes) (on_board yes) (dnp no) (fields_autoplaced)
-    (property "Reference" "U1" (at 86.0141 17.78 0)
-      (effects (font (size 1.27 1.27)) (justify left))
-    )
-    (property "Value" "ESP32-S3-WROOM-1-N16R8" (at 86.0141 20.32 0)
-      (effects (font (size 1.27 1.27)) (justify left))
-    )
-    (property "Footprint" "Espressif:ESP32-S3-WROOM-1" (at 86.36 109.22 0)
-      (effects (font (size 1.27 1.27)) hide)
-    )
-    (property "Datasheet" "https://www.espressif.com/sites/default/files/documentation/esp32-s3-wroom-1_wroom-1u_datasheet_en.pdf" (at 86.36 111.76 0)
-      (effects (font (size 1.27 1.27)) hide)
-    )
-    (property "JLCPCB Part" "C2913202" (at 83.82 60.96 0)
+  (symbol (lib_id "mantyl:ESP32-S3-WROOM-1") (at 138.43 64.77 0) (unit 1)
+    (in_bom yes) (on_board yes) (dnp no) (fields_autoplaced)
+    (property "Reference" "U1" (at 140.6241 21.59 0)
+      (effects (font (size 1.27 1.27)) (justify left))
+    )
+    (property "Value" "ESP32-S3-WROOM-1-N16R8" (at 140.6241 24.13 0)
+      (effects (font (size 1.27 1.27)) (justify left))
+    )
+    (property "Footprint" "Espressif:ESP32-S3-WROOM-1" (at 140.97 129.54 0)
+      (effects (font (size 1.27 1.27)) hide)
+    )
+    (property "Datasheet" "https://www.espressif.com/sites/default/files/documentation/esp32-s3-wroom-1_wroom-1u_datasheet_en.pdf" (at 140.97 132.08 0)
+      (effects (font (size 1.27 1.27)) hide)
+    )
+    (property "JLCPCB Part" "C2913202" (at 138.43 64.77 0)
       (effects (font (size 1.27 1.27)) hide)
     )
@@
     (pin "39")
     (pin "4")
-    (pin "40")
-    (pin "41")
     (pin "5")
     (pin "6")
@@
     (pin "8")
     (pin "9")
+    (pin "40")
+    (pin "41")
     (instances
       (project "v2_numpad"
@@
         )
       )
+    )
+  )
+  (symbol (lib_id "power:GND") (at 48.26 46.99 0) (unit 1)
+    (in_bom yes) (on_board yes) (dnp no) (fields_autoplaced)
+    (property "Reference" "#PWR05" (at 48.26 53.34 0)
+      (effects (font (size 1.27 1.27)) hide)
+    )
+    (property "Value" "GND" (at 48.26 52.07 0)
+      (effects (font (size 1.27 1.27)))
+    )
+    (property "Footprint" "" (at 48.26 46.99 0)
+      (effects (font (size 1.27 1.27)) hide)
+    )
+    (property "Datasheet" "" (at 48.26 46.99 0)
+      (effects (font (size 1.27 1.27)) hide)
+    )
+    (pin "1")
+    (instances
+      (project "v2_numpad"
+        (path "/42eee74c-d04d-4a1d-8e02-a7aca1694734/74c564bf-cb18-45a0-a3d5-47831683800e"
+          (reference "#PWR05") (unit 1)
+        )
+      )
