File: kicad/esp32s3/usb.kicad_sch (KiCad schematic)
At the start: 33 parts, among them J1 USB_C_Receptacle_USB2.0, J2 USB_C_Receptacle_USB2.0, Q1 S8050, Q2 S8050, SW1 SW_MEC_5E, SW2 SW_MEC_5E, U2 USBLC6-2P6, U3 USBLC6-2P6, U4 AMS1117-3.3, U5 CP2102N-Axx-xQFN24

Commit message: [kicad] update annotations in esp32s3 template
Parts:
- renumbered R9 to R10, R10 to R11, R11 to R12, R12 to R13, R4 to R3, R3 to R4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
